Commit message: changing the ability hand filenames and urdfs to be compatible with IsaacLabs USD transfer tool

File: robots/assembly/xarm7_ability/xarm7_ability_right_hand.urdf (robot description, URDF)
Before this commit: robot xarm7_ability_right, 26 links, 25 joints
Links:
- link base: geometry collision mesh filename=/home/joao-marques/dexmate/dexmate_take_home/dex-urdf/robot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; visual mesh filename=/home/joao-marques/dexmate/dexmate_take_home/dex-urdf/robot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
- link index_L1: geometry collision box size=0.012 0.012 0.002; collision box size=0.012 0.012 0.002
- link index_L2: geometry collision mesh filename=/home/joao-marques/dexmate/dexmate_take_home/dex-urdf/robot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; collision sphere radius=0.007
- link link1: geometry collision mesh filename=/home/joao-marques/dexmate/dexmate_take_home/dex-urdf/robot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; visual mesh filename=/home/joao-marques/dexmate/dexmate_take_home/dex-urdf/robot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
- link link2: geometry collision mesh filename=/home/joao-marques/dexmate/dexmate_take_home/dex-urdf/robot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; visual mesh filename=/home/joao-marques/dexmate/dexmate_take_home/dex-urdf/robot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
- link link3: geometry collision mesh filename=/home/joao-marques/dexmate/dexmate_take_home/dex-urdf/robot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; visual mesh filename=/home/joao-marques/dexmate/dexmate_take_home/dex-urdf/robot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
- link link4: geometry collision mesh filename=/home/joao-marques/dexmate/dexmate_take_home/dex-urdf/robot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; visual mesh filename=/home/joao-marques/dexmate/dexmate_take_home/dex-urdf/robot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
- link link5: geometry collision mesh filename=/home/joao-marques/dexmate/dexmate_take_home/dex-urdf/robot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; visual mesh filename=/home/joao-marques/dexmate/dexmate_take_home/dex-urdf/robot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
- link link6: geometry collision mesh filename=/home/joao-marques/dexmate/dexmate_take_home/dex-urdf/robot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; visual mesh filename=/home/joao-marques/dexmate/dexmate_take_home/dex-urdf/robot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
- link link7: geometry collision cylinder length=0.018 radius=0.0365; collision mesh filename=/home/joao-marques/dexmate/dexmate_take_home/dex-urdf/robot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
- link link_base: geometry collision mesh filename=/home/joao-marques/dexmate/dexmate_take_home/dex-urdf/robot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; visual mesh filename=/home/joao-marques/dexmate/dexmate_take_home/dex-urdf/robot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
- link middle_L1: geometry collision box size=0.012 0.012 0.002; collision box size=0.012 0.012 0.002
- link middle_L2: geometry collision mesh filename=/home/joao-marques/dexmate/dexmate_take_home/dex-urdf/robot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; collision sphere radius=0.007
- link pinky_L1: geometry collision box size=0.012 0.012 0.002; collision box size=0.012 0.012 0.002
- link pinky_L2: geometry collision mesh filename=/home/joao-marques/dexmate/dexmate_take_home/dex-urdf/robot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; collision sphere radius=0.007
- link ring_L1: geometry collision box size=0.012 0.012 0.002; collision box size=0.012 0.012 0.002
- link ring_L2: geometry collision mesh filename=/home/joao-marques/dexmate/dexmate_take_home/dex-urdf/robot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; collision sphere radius=0.007
- link thumb_L1: geometry collision mesh filename=/home/joao-marques/dexmate/dexmate_take_home/dex-urdf/robot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; visual mesh filename=/home/joao-marques/dexmate/dexmate_take_home/dex-urdf/robot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
- link thumb_L2: geometry collision mesh filename=/home/joao-marques/dexmate/dexmate_take_home/dex-urdf/robot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; visual mesh filename=/home/joao-marques/dexmate/dexmate_take_home/dex-urdf/robot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
- link thumb_base: geometry collision mesh filename=/home/joao-marques/dexmate/dexmate_take_home/dex-urdf/robot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; visual mesh filename=/home/joao-marques/dexmate/dexmate_take_home/dex-urdf/robot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
